File: pcb/GLaDOS-Cam/GLaDOS-Cam.kicad_pcb (KiCad board)
At the start: 2 copper layers, 100 x 100 mm, 11 parts, among them U1 STM32U575VIT6, U2 IS66WVH8M8BLL-100B1LI, U3 STLQ020C33R, U4 STLQ020C33R, U5 XC6206-2_8V, U6 XC6206-1_2V_C49446790, U7 FH12-24S-0_5SH(55), U8 TF-CARD_H1_8, U9 TS-1187A-B-A-B, X1 X322516MLB4SI

Commit message: Push local devs
Parts:
- added J1: Conn_01x03_Socket, Connector_PinSocket_2.54mm:PinSocket_1x03_P2.54mm_Vertical, F.Cu at (149.1, 80.0)
- added J2: Conn_01x03_Socket, Connector_PinSocket_2.54mm:PinSocket_1x03_P2.54mm_Vertical, F.Cu at (153.7, 80.0)

Commit message: Push local devs
Parts:
- added C1: 9pF, Capacitor_SMD:C_0603_1608Metric_Pad1.08x0.95mm_HandSolder, F.Cu at (146.2, 101.8)
- added C10: 10uF, Capacitor_SMD:C_0603_1608Metric_Pad1.08x0.95mm_HandSolder, F.Cu at (150.6, 109.3)
- added C11: 100nF, Capacitor_SMD:C_0603_1608Metric_Pad1.08x0.95mm_HandSolder, F.Cu at (150.6, 111.8)
- added C12: 10uF, Capacitor_SMD:C_0603_1608Metric_Pad1.08x0.95mm_HandSolder, F.Cu at (150.6, 114.3)
- added C13: 100nF, Capacitor_SMD:C_0603_1608Metric_Pad1.08x0.95mm_HandSolder, F.Cu at (154.9, 101.8)
- added C14: 10uF, Capacitor_SMD:C_0603_1608Metric_Pad1.08x0.95mm_HandSolder, F.Cu at (154.9, 104.3)
- added C15: 100nF, Capacitor_SMD:C_0603_1608Metric_Pad1.08x0.95mm_HandSolder, F.Cu at (154.9, 106.8)
- added C16: 10uF, Capacitor_SMD:C_0603_1608Metric_Pad1.08x0.95mm_HandSolder, F.Cu at (154.9, 109.3)
- added C17: 100nF, Capacitor_SMD:C_0603_1608Metric_Pad1.08x0.95mm_HandSolder, F.Cu at (154.9, 111.8)
- added C18: 10uF, Capacitor_SMD:C_0603_1608Metric_Pad1.08x0.95mm_HandSolder, F.Cu at (154.9, 114.3)
- added C19: 4.7uF, Capacitor_SMD:C_0603_1608Metric_Pad1.08x0.95mm_HandSolder, F.Cu at (159.3, 101.8)
- added C2: 9pF, Capacitor_SMD:C_0603_1608Metric_Pad1.08x0.95mm_HandSolder, F.Cu at (146.2, 104.3)
- added C20: 100nF, Capacitor_SMD:C_0603_1608Metric_Pad1.08x0.95mm_HandSolder, F.Cu at (159.3, 104.3)
- added C21: 10uF, Capacitor_SMD:C_0603_1608Metric_Pad1.08x0.95mm_HandSolder, F.Cu at (159.3, 106.8)
- added C22: 100nF, Capacitor_SMD:C_0603_1608Metric_Pad1.08x0.95mm_HandSolder, F.Cu at (159.3, 109.3)
- added C23: 100nF, Capacitor_SMD:C_0603_1608Metric_Pad1.08x0.95mm_HandSolder, F.Cu at (159.3, 111.8)
- added C3: 9pF, Capacitor_SMD:C_0603_1608Metric_Pad1.08x0.95mm_HandSolder, F.Cu at (146.2, 106.8)
- added C4: 9pF, Capacitor_SMD:C_0603_1608Metric_Pad1.08x0.95mm_HandSolder, F.Cu at (146.2, 109.3)
- added C5: 100nF, Capacitor_SMD:C_0603_1608Metric_Pad1.08x0.95mm_HandSolder, F.Cu at (146.2, 111.8)
- added C6: 10uF, Capacitor_SMD:C_0603_1608Metric_Pad1.08x0.95mm_HandSolder, F.Cu at (146.2, 114.3)
- added C7: 100nF, Capacitor_SMD:C_0603_1608Metric_Pad1.08x0.95mm_HandSolder, F.Cu at (150.6, 101.8)
- added C8: 10uF, Capacitor_SMD:C_0603_1608Metric_Pad1.08x0.95mm_HandSolder, F.Cu at (150.6, 104.3)
- added C9: 100nF, Capacitor_SMD:C_0603_1608Metric_Pad1.08x0.95mm_HandSolder, F.Cu at (150.6, 106.8)
- added R1: R, Resistor_SMD:R_0603_1608Metric_Pad0.98x0.95mm_HandSolder, F.Cu at (159.3, 114.3)
- added U10: TS-1187A-B-A-B, glados-cam-lib:SW-SMD_4P-L5.1-W5.1-P3.70-LS6.5-TL_H1.5, F.Cu at (148.1, 118.8)
Connections:
- TXAL1 pad 1: unconnected-(TXAL1-Pad1) -> /MCU/XTAL_32K_1
- TXAL1 pad 2: unconnected-(TXAL1-Pad2) -> /MCU/XTAL_32K_2
- U1 pad 10: unconnected-(U1-VSS-Pad10) -> GND
- U1 pad 100: unconnected-(U1-VDD-Pad100) -> +3.3V
- U1 pad 11: unconnected-(U1-VDD-Pad11) -> +3.3V
- U1 pad 12: unconnected-(U1-OSC_IN-PF0-Pad12) -> /MCU/XTAL_16M_1
- U1 pad 13: unconnected-(U1-OSC_OUT-PF1-Pad13) -> /MCU/XTAL_16M_2
- U1 pad 14: unconnected-(U1-NRST-Pad14) -> /MCU/NRST
- U1 pad 19: unconnected-(U1-VSSA-Pad19) -> GND
- U1 pad 20: unconnected-(U1-VREF--Pad20) -> GND
- U1 pad 21: unconnected-(U1-VREF+-Pad21) -> +3.3V
- U1 pad 22: unconnected-(U1-VDDA-Pad22) -> +3.3V
- U1 pad 27: unconnected-(U1-VSS-Pad27) -> GND
- U1 pad 28: unconnected-(U1-VDD-Pad28) -> +3.3V
- U1 pad 48: unconnected-(U1-VCAP-Pad48) -> /MCU/VCAP
- U1 pad 49: unconnected-(U1-VSS-Pad49) -> GND
- U1 pad 50: unconnected-(U1-VDD-Pad50) -> +3.3V
- U1 pad 6: unconnected-(U1-VBAT-Pad6) -> +3.3V
- U1 pad 73: unconnected-(U1-VDDUSB-Pad73) -> VBUS
- U1 pad 74: unconnected-(U1-VSS-Pad74) -> GND
- U1 pad 75: unconnected-(U1-VDD-Pad75) -> +3.3V
- U1 pad 8: unconnected-(U1-OSC32_IN-PC14-Pad8) -> /MCU/XTAL_32K_1
- U1 pad 9: unconnected-(U1-OSC32_OUT-PC15-Pad9) -> /MCU/XTAL_32K_2
- U1 pad 94: unconnected-(U1-PH3-BOOTO-Pad94) -> /MCU/BOOT0
- U1 pad 99: unconnected-(U1-VSS-Pad99) -> GND
- U9 pad 1: unconnected-(U9-A-Pad1) -> /MCU/NRST
- U9 pad 2: unconnected-(U9-B-Pad2) -> Net-(U9-B)
- U9 pad 3: unconnected-(U9-C-Pad3) -> GND
- U9 pad 4: unconnected-(U9-D-Pad4) -> GND
- X1 pad 1: unconnected-(X1-OSC1-Pad1) -> /MCU/XTAL_16M_1
- X1 pad 2: unconnected-(X1-GND-Pad2) -> GND
- X1 pad 3: unconnected-(X1-OSC2-Pad3) -> /MCU/XTAL_16M_2
- X1 pad 4: unconnected-(X1-GND-Pad4) -> GND
