File: pcb/GLaDOS-Cam/mcu.kicad_sch (KiCad schematic)
At the start: 4 parts, among them U1 STM32U575VIT6, U9 TS-1187A-B-A-B, X1 X322516MLB4SI

Commit message: Push local devs
Parts:
- added C1, C2, C3, C4: 9pF, Capacitor_SMD:C_0603_1608Metric_Pad1.08x0.95mm_HandSolder, symbol Device:C
- added C10, C12, C14, C16, C18, C21, C6, C8: 10uF, Capacitor_SMD:C_0603_1608Metric_Pad1.08x0.95mm_HandSolder, symbol Device:C
- added C11, C13, C15, C17, C20, C22, C23, C5, C7, C9: 100nF, Capacitor_SMD:C_0603_1608Metric_Pad1.08x0.95mm_HandSolder, symbol Device:C
- added C19: 4.7uF, Capacitor_SMD:C_0603_1608Metric_Pad1.08x0.95mm_HandSolder, symbol Device:C
- added R1: R, Resistor_SMD:R_0603_1608Metric_Pad0.98x0.95mm_HandSolder, symbol Device:R
- added U10: TS-1187A-B-A-B, glados-cam-lib:SW-SMD_4P-L5.1-W5.1-P3.70-LS6.5-TL_H1.5, symbol glados-cam-lib:TS-1187A-B-A-B
Connections:
- net XTAL_32K_1: now reaches TXAL1.1
- net XTAL_32K_1: now also U1.8 (OSC32_IN-PC14), C3.1
- net XTAL_32K_2: now reaches TXAL1.2
- net XTAL_32K_2: now also U1.9 (OSC32_OUT-PC15), C4.1
- net GND: now reaches U1.10 (VSS)
- net GND: now also U1.19 (VSSA), U1.20 (VREF-), U1.27 (VSS), U1.49 (VSS), U1.74 (VSS), U1.99 (VSS), U9.3 (C), U9.4 (D), X1.2 (GND), X1.4 (GND), C1.2, C10.2, C11.2, C12.2, C13.2, C14.2, C15.2, C16.2, C17.2, C18.2, C19.2, C2.2, C20.2, C21.2, C22.2, C3.2, C4.2, C5.2, C6.2, C7.2, C8.2, C9.2, R1.2
- net +3.3V: now reaches U1.100 (VDD)
- net +3.3V: now also U1.11 (VDD), U1.21 (VREF+), U1.22 (VDDA), U1.28 (VDD), U1.50 (VDD), U1.6 (VBAT), U1.75 (VDD), C10.1, C11.1, C12.1, C13.1, C14.1, C15.1, C16.1, C17.1, C18.1, C20.1, C21.1, C23.1, C5.1, C6.1, C7.1, C8.1, C9.1, U10.1 (A), U10.2 (B)
- net XTAL_16M_1: now reaches U1.12 (OSC_IN-PF0)
- net XTAL_16M_1: now also X1.1 (OSC1), C1.1
- net XTAL_16M_2: now reaches U1.13 (OSC_OUT-PF1)
- net XTAL_16M_2: now also X1.3 (OSC2), C2.1
- net NRST: now reaches U1.14 (NRST)
- net NRST: now also U9.1 (A)
- net VCAP: now reaches U1.48 (VCAP)
- net VCAP: now also C19.1
- net VBUS: now reaches U1.73 (VDDUSB)
- net BOOT0: now reaches U1.94 (PH3-BOOTO)
- net BOOT0: now also R1.1, U10.3 (C)
- net at U9.2 (B): now also C22.1
- new net: C23.2, U10.4 (D)
Other:
- moved on the sheet: TXAL1, U9, X1
