File: pcb/GLaDOS-Cam/power.kicad_sch (KiCad schematic)
At the start: 4 parts, among them U3 STLQ020C33R, U4 STLQ020C33R, U5 XC6206-2_8V, U6 XC6206-1_2V_C49446790

Commit message: Push local devs
Other:
- moved on the sheet: U4, U6
Changed lines of the file:
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@@
 	(symbol
 		(lib_id "glados-cam-lib:STLQ020C33R")
-		(at 137.16 102.87 0)
+		(at 140.97 115.57 0)
 		(unit 1)
 		(exclude_from_sim no)
@@
 		(fields_autoplaced yes)
 		(property "Reference" "U4"
-			(at 137.16 92.71 0)
+			(at 140.97 105.41 0)
 			(effects
 				(font
@@
 		)
 		(property "Value" "STLQ020C33R"
-			(at 137.16 95.25 0)
+			(at 140.97 107.95 0)
 			(effects
 				(font
@@
 		)
 		(property "Footprint" "glados-cam-lib:TSSOP-5_L2.0-W1.3-P0.65-LS2.1-BL"
-			(at 137.16 113.03 0)
+			(at 140.97 125.73 0)
 			(effects
 				(font
@@
 		)
 		(property "Datasheet" "https://atta.szlcsc.com/upload/public/pdf/source/20171208/C152728_15127341294501171490.pdf"
-			(at 134.874 102.743 0)
+			(at 138.684 115.443 0)
 			(effects
 				(font
@@
 		)
 		(property "Description" ""
-			(at 137.16 102.87 0)
+			(at 140.97 115.57 0)
 			(effects
 				(font
@@
 		)
 		(property "LCSC" "C2970558"
-			(at 137.16 102.87 0)
+			(at 140.97 115.57 0)
 			(effects
 				(font
@@
 	(symbol
 		(lib_id "glados-cam-lib:XC6206-1_2V_C49446790")
-		(at 212.09 107.95 0)
+		(at 215.9 120.65 0)
 		(unit 1)
 		(exclude_from_sim no)
@@
 		(fields_autoplaced yes)
 		(property "Reference" "U6"
-			(at 212.09 99.06 0)
+			(at 215.9 111.76 0)
 			(effects
 				(font
@@
 		)
 		(property "Value" "XC6206-1_2V_C49446790"
-			(at 212.09 101.6 0)
+			(at 215.9 114.3 0)
 			(effects
 				(font
@@
 		)
 		(property "Footprint" "glados-cam-lib:SOT-23-3_L3.0-W1.6-P1.90-LS2.8-BR"
-			(at 212.09 118.11 0)
+			(at 215.9 130.81 0)
 			(effects
 				(font
@@
 		)
 		(property "Datasheet" "https://atta.szlcsc.com/upload/public/pdf/source/20200309/C150720_EA5FFAC42CC5D7D051BA246B6393078B.pdf"
-			(at 209.804 107.823 0)
+			(at 213.614 120.523 0)
 			(effects
 				(font
@@
 		)
 		(property "Description" ""
-			(at 212.09 107.95 0)
+			(at 215.9 120.65 0)
 			(effects
 				(font
@@
 		)
 		(property "LCSC" "C49446790"
-			(at 212.09 107.95 0)
-			(effects
-				(font
+			(at 215.9 120.65 0)
+			(effects
+				(font
